File: differential/WolfDrive_encoder_renishaw_adapter.sch (KiCad schematic (older format))
At the start: 18 parts, among them CN1 SPI/BiSS, CN2 Conn_01x10_Female, U1 AP131-33, U2 TPD8F003

Commit message: Library fix for KiCAD v5, changed differential drivers to RS485 compatible
Parts:
- removed I1: DS90LV027A, Housings_SOIC:SOIC-8_3.9x4.9mm_Pitch1.27mm, symbol DriveSymbols:DS90LV027A
- removed I2: DS90LV028A, Housings_SOIC:SOIC-8_3.9x4.9mm_Pitch1.27mm, symbol DriveSymbols:DS90LV028A
- added U? (x2): UA9638CD, Package_SO:SOIC-8_3.9x4.9mm_P1.27mm, symbol Interface_LineDriver:UA9638CD
- added U? (x2): UA9637, Package_DIP:DIP-8_W7.62mm, symbol Interface_LineDriver:UA9637
- C1, C2, C3, C4, C5, C7: symbol device:C_Small -> Device:C_Small
- CN2: symbol conn:Conn_01x10_Female -> Connector:Conn_01x10_Female
- D1: symbol device:D_TVS -> Device:D_TVS
- MK1, MK2, MK3: symbol mechanical:Mounting_Hole_PAD -> Mechanical:Mounting_Hole_PAD
- R1, R2: symbol device:R -> Device:R
- U1: symbol regul:AP131-33 -> Regulator_Linear:AP131-33
- U2: symbol ESD_Protection:TPD8F003 -> Power_Protection:TPD8F003
Connections:
- wire segments 42 -> 39
